File: kicad/env.sch (KiCad schematic (older format))
At the start: 24 parts, among them Q1 2SC1740SQ, Q2 2SC1740SQ, Q3 2SC1740SQ

Commit message: a
Parts:
- removed D35: 1SS254, symbol pspice:DIODE
- added D35: 1SS254, symbol Device:D
- C1, C2, C4: symbol pspice:C -> Device:C
- C3: symbol pspice:C -> Device:CP
- D33, D34: symbol pspice:DIODE -> Device:D
- Q1, Q2, Q3: symbol pspice:QNPN -> Device:Q_NPN_CBE
- R1, R10, R11, R12, R13, R14, R2, R3, R4, R5, R6, R7, R8, R9: symbol pspice:R -> Device:R
Connections:
- wire segments 64 -> 69
Other:
- note removed: "+"
