File: kicad/env.sch (KiCad schematic (older format))
At the start: 24 parts, among them Q1 2SC1740SQ, Q2 2SC1740SQ, Q3 2SC1740SQ

Commit message: 'a'
Connections:
- net ES renamed ENV
- net OUTPUT renamed OUT
- net PS renamed PITCH
