File: kicad/digital.sch (KiCad schematic (older format))
At the start: 6 parts

Commit message: a
Parts:
- added U?: D4168C, symbol parts:D4168C
Connections:
- net A13: now also U?.26 (A13)
- net A0: now reaches U?.10 (A0)
- net D0: now reaches U?.11 (D0)
- net D1: now reaches U?.12 (D1)
- net D2: now reaches U?.13 (D2)
- net D3: now reaches U?.15 (D3)
- net D4: now reaches U?.16 (D4)
- net D5: now reaches U?.17 (D5)
- net D6: now reaches U?.18 (D6)
- net D7: now reaches U?.19 (D7)
- net A12: now reaches U?.2 (A12)
- net A10: now reaches U?.21 (A10)
- net A11: now reaches U?.23 (A11)
- net A9: now reaches U?.24 (A9)
- net A8: now reaches U?.25 (A8)
- net A14: now reaches U?.27 (A14)
- net A7: now reaches U?.3 (A7)
- net A6: now reaches U?.4 (A6)
- net A5: now reaches U?.5 (A5)
- net A4: now reaches U?.6 (A4)
- net A3: now reaches U?.7 (A3)
- net A2: now reaches U?.8 (A2)
- net A1: now reaches U?.9 (A1)
- no-connect marks 1 -> 0
Other:
- moved on the sheet: U?
Changed lines of the file:
@@
 $EndDescr
-$Comp
-L Memory_EPROM:27C256 U?
-U 1 1 5F82BB6B
-P 9850 4300
-F 0 "U?" H 9850 5581 50  0000 C CNN
-F 1 "27C256" H 9850 5490 50  0000 C CNN
-F 2 "Package_DIP:DIP-28_W15.24mm" H 9850 4300 50  0001 C CNN
-F 3 "http://ww1.microchip.com/downloads/en/DeviceDoc/doc0014.pdf" H 9850 4300 50  0001 C CNN
-	1    9850 4300
-	1    0    0    -1
-$EndComp
 $Comp
 L 74xx:74HC02 U?
@@
 Wire Wire Line
 	5650 1550 6550 1550
-NoConn ~ 10250 5050
+$Comp
+L parts:D4168C U?
+U 1 1 5F83BA0D
+P 7700 4100
+F 0 "U?" H 7750 5031 50  0000 C CNN
+F 1 "D4168C" H 7750 4940 50  0000 C CNN
+F 2 "" H 7700 4100 50  0001 C CNN
+F 3 "" H 7700 4100 50  0001 C CNN
+	1    7700 4100
+	1    0    0    -1
+$EndComp
+$Comp
+L Memory_EPROM:27C256 U?
+U 1 1 5F82BB6B
+P 10100 4300
+F 0 "U?" H 10100 5581 50  0000 C CNN
+F 1 "27C256" H 10100 5490 50  0000 C CNN
+F 2 "Package_DIP:DIP-28_W15.24mm" H 10100 4300 50  0001 C CNN
+F 3 "http://ww1.microchip.com/downloads/en/DeviceDoc/doc0014.pdf" H 10100 4300 50  0001 C CNN
+	1    10100 4300
+	1    0    0    -1
+$EndComp
+Entry Wire Line
+	9450 3300 9550 3400
+Entry Wire Line
+	9450 3400 9550 3500
+Entry Wire Line
+	9450 3500 9550 3600
+Entry Wire Line
+	9450 3600 9550 3700
+Entry Wire Line
+	9450 3800 9550 3900
+Entry Wire Line
+	9450 3700 9550 3800
+Entry Wire Line
+	9450 3900 9550 4000
+Entry Wire Line
+	9450 4000 9550 4100
+Entry Wire Line
+	9450 4100 9550 4200
+Entry Wire Line
+	9450 4200 9550 4300
+Entry Wire Line
+	9450 4300 9550 4400
+Entry Wire Line
+	9450 4500 9550 4600
+Entry Wire Line
+	9450 4400 9550 4500
+Entry Wire Line
+	9450 4700 9550 4800
+Entry Wire Line
+	9450 4600 9550 4700
+Wire Wire Line
+	10500 3400 10600 3400
+Wire Wire Line
+	10500 3500 10600 3500
+Wire Wire Line
+	10500 3600 10600 3600
+Wire Wire Line
+	10500 3700 10600 3700
+Wire Wire Line
+	10500 3800 10600 3800
+Wire Wire Line
+	10500 3900 10600 3900
+Wire Wire Line
+	10500 4000 10600 4000
+Wire Wire Line
+	10500 4100 10600 4100
+Entry Wire Line
+	10600 3400 10700 3500
+Entry Wire Line
+	10600 3500 10700 3600
+Entry Wire Line
+	10600 3600 10700 3700
+Entry Wire Line
+	10600 3700 10700 3800
+Entry Wire Line
+	10600 3800 10700 3900
+Entry Wire Line
+	10600 3900 10700 4000
+Entry Wire Line
+	10600 4000 10700 4100
+Entry Wire Line
+	10600 4100 10700 4200
+Text Label 9550 3400 0    50   ~ 0
+A0
+Text Label 9550 3500 0    50   ~ 0
+A1
+Text Label 9550 3600 0    50   ~ 0
+A2
+Text Label 9550 3700 0    50   ~ 0
+A3
+Text Label 9550 3800 0    50   ~ 0
+A4
+Text Label 9550 3900 0    50   ~ 0
+A5
+Text Label 9550 4000 0    50   ~ 0
+A6
+Text Label 9550 4100 0    50   ~ 0
+A7
+Text Label 9550 4200 0    50   ~ 0
+A8
+Text Label 9550 4300 0    50   ~ 0
+A9
+Text Label 9550 4400 0    50   ~ 0
+A10
+Text Label 9550 4500 0    50   ~ 0
+A11
+Text Label 9550 4600 0    50   ~ 0
+A12
+Text Label 9550 4700 0    50   ~ 0
+A13
+Text Label 9550 4800 0    50   ~ 0
+A14
+Wire Wire Line
+	9550 3400 9700 3400
+Wire Wire Line
+	9550 3500 9700 3500
+Wire Wire Line
+	9550 3600 9700 3600
+Wire Wire Line
+	9550 3700 9700 3700
+Wire Wire Line
+	9550 3800 9700 3800
+Wire Wire Line
+	9550 3900 9700 3900
+Wire Wire Line
+	9550 4000 9700 4000
+Wire Wire Line
+	9550 4100 9700 4100
+Wire Wire Line
+	9550 4200 9700 4200
+Wire Wire Line
+	9550 4300 9700 4300
+Wire Wire Line
+	9550 4400 9700 4400
+Wire Wire Line
+	9550 4500 9700 4500
+Wire Wire Line
+	9550 4600 9700 4600
+Wire Wire Line
+	9550 4700 9700 4700
+Wire Wire Line
+	9550 4800 9700 4800
+Text Label 10500 3400 0    50   ~ 0
+D0
+Text Label 10500 3500 0    50   ~ 0
+D1
+Text Label 10500 3600 0    50   ~ 0
+D2
+Text Label 10500 3700 0    50   ~ 0
+D3
+Text Label 10500 3800 0    50   ~ 0
+D4
+Text Label 10500 3900 0    50   ~ 0
+D5
+Text Label 10500 4000 0    50   ~ 0
+D6
+Text Label 10500 4100 0    50   ~ 0
+D7
+Wire Bus Line
+	10700 3500 10700 5650
+Wire Bus Line
+	9450 3300 9450 4700
 $EndSCHEMATC

Commit message: a
Parts:
- removed U?: D4168C, symbol parts:D4168C
- added U? (x2): D4168C, symbol parts:D4168C
Connections:
- net A0: now also U?.10 (A0), U?.10 (A0)
- net A1: now also U?.9 (A1), U?.9 (A1)
- net A10: now also U?.21 (A10), U?.21 (A10)
- net A11: now also U?.23 (A11), U?.23 (A11)
- net A12: now also U?.2 (A12), U?.2 (A12)
- net A2: now also U?.8 (A2), U?.8 (A2)
- net A3: now also U?.7 (A3), U?.7 (A3)
- net A4: now also U?.6 (A4), U?.6 (A4)
- net A5: now also U?.5 (A5), U?.5 (A5)
- net A6: now also U?.4 (A6), U?.4 (A6)
- net A7: now also U?.3 (A7), U?.3 (A7)
- net A8: now also U?.25 (A8), U?.25 (A8)
- net A9: now also U?.24 (A9), U?.24 (A9)
- net D0: now also U?.11 (D0), U?.11 (D0)
- net D1: now also U?.12 (D1), U?.12 (D1)
- net D2: now also U?.13 (D2), U?.13 (D2)
- net D3: now also U?.15 (D3), U?.15 (D3)
- net D4: now also U?.16 (D4), U?.16 (D4)
- net D5: now also U?.17 (D5), U?.17 (D5)
- net D6: now also U?.18 (D6), U?.18 (D6)
- net D7: now also U?.19 (D7), U?.19 (D7)

Commit message: a
Parts:
- added C? (x3): 100nF, symbol Device:C
- added C?: 10uF @ 16V, symbol Device:CP
Connections:
- net VL2: now reaches U?.14 (GND)
- net VL2: now also U?.14 (GND), U?.14 (GND), C?.1, C?.1, C?.1, C?.2
- net at U?.20 (~CE): now also U?.20 (~CE), U?.20 (~CE)
- net VA: now reaches U?.28 (VCC)
- net VA: now also U?.28 (VCC), U?.28 (VCC), C?.1, C?.2, C?.2, C?.2
- net at U?.1 (~RFSH): now also U?.1 (~RFSH)
- net at U?.22 (~OE): now also U?.22 (~OE)
- net at U?.27 (~WE): now also U?.27 (~WE)
- no-connect marks 0 -> 1
Other:
- moved on the sheet: U?

Commit message: cleanup
Connections:
- net VL2: now also U?.1 (~RFSH), U?.1 (~RFSH)
Other:
- moved on the sheet: C?, U?

Commit message: oki
Parts:
- added U?: MSM6283, symbol parts:MSM6283
Connections:
- net A15: now also U?.22 (~OE)
- net at U?.20 (~CE), U?.20 (~CE), U?.20 (~CE): now also U?.15 (~CE)
- net at U?.1: now also U?.26 (CS)
- net at U?.13: now also U?.26 (CS)
- net at U?.22 (~OE), U?.22 (~OE): now also U?.19 (~OE)
- net at U?.27 (~WE), U?.27 (~WE): now also U?.31 (~WE)
Changed lines of the file:
@@
 	10650 4600 10750 4600
 Entry Wire Line
-	10750 3900 10850 4000
-Entry Wire Line
-	10750 4000 10850 4100
-Entry Wire Line
-	10750 4100 10850 4200
-Entry Wire Line
-	10750 4200 10850 4300
-Entry Wire Line
-	10750 4300 10850 4400
-Entry Wire Line
-	10750 4400 10850 4500
-Entry Wire Line
-	10750 4500 10850 4600
-Entry Wire Line
-	10750 4600 10850 4700
+	10750 4000 10850 3900
+Entry Wire Line
+	10750 4100 10850 4000
+Entry Wire Line
+	10750 4200 10850 4100
+Entry Wire Line
+	10750 4300 10850 4200
+Entry Wire Line
+	10750 4400 10850 4300
+Entry Wire Line
+	10750 4500 10850 4400
+Entry Wire Line
+	10750 4600 10850 4500
+Entry Wire Line
+	10750 3900 10850 3800
 Text Label 9700 3900 0    50   ~ 0
 A0
@@
 Text Label 10650 4600 0    50   ~ 0
 D7
-Wire Bus Line
-	10850 3450 9600 3450
 Wire Wire Line
 	9200 4100 9300 4100
@@
 D7
 Entry Wire Line
-	9300 4100 9400 4200
-Entry Wire Line
-	9300 4200 9400 4300
-Entry Wire Line
-	9300 4300 9400 4400
-Entry Wire Line
-	9300 4400 9400 4500
-Entry Wire Line
-	9300 4500 9400 4600
-Entry Wire Line
-	9300 4600 9400 4700
-Entry Wire Line
-	9300 4700 9400 4800
-Entry Wire Line
-	9300 4800 9400 4900
-Connection ~ 9600 3450
+	9300 4200 9400 4100
+Entry Wire Line
+	9300 4300 9400 4200
+Entry Wire Line
+	9300 4400 9400 4300
+Entry Wire Line
+	9300 4500 9400 4400
+Entry Wire Line
+	9300 4600 9400 4500
+Entry Wire Line
+	9300 4700 9400 4600
+Entry Wire Line
+	9300 4800 9400 4700
+Entry Wire Line
+	9300 4100 9400 4000
 Wire Wire Line
 	8400 4100 8250 4100
@@
 Entry Wire Line
 	8150 5200 8250 5300
-Wire Bus Line
-	8150 3450 9400 3450
 Wire Wire Line
 	7750 4100 7850 4100
@@
 Text Label 7750 4100 0    50   ~ 0
 D0
-Text Label 7750 4200 0    50   ~ 0
-D1
 Text Label 7750 4300 0    50   ~ 0
 D2
@@
 D7
 Entry Wire Line
-	7850 4100 7950 4200
-Entry Wire Line
-	7850 4200 7950 4300
-Entry Wire Line
-	7850 4300 7950 4400
-Entry Wire Line
-	7850 4400 7950 4500
-Entry Wire Line
-	7850 4500 7950 4600
-Entry Wire Line
-	7850 4600 7950 4700
-Entry Wire Line
-	7850 4700 7950 4800
-Entry Wire Line
-	7850 4800 7950 4900
+	7850 4200 7950 4100
+Entry Wire Line
+	7850 4300 7950 4200
+Entry Wire Line
+	7850 4400 7950 4300
+Entry Wire Line
+	7850 4500 7950 4400
+Entry Wire Line
+	7850 4600 7950 4500
+Entry Wire Line
+	7850 4700 7950 4600
+Entry Wire Line
+	7850 4800 7950 4700
+Entry Wire Line
+	7850 4100 7950 4000
 Wire Wire Line
 	6950 4100 6800 4100
@@
 Entry Wire Line
 	6700 5200 6800 5300
-Wire Bus Line
-	6700 3450 7950 3450
 Connection ~ 8150 3450
 Text Label 6800 6000 0    50   ~ 0
@@
 Connection ~ 8800 6000
 Wire Wire Line
-	9400 5600 9850 5600
-Connection ~ 9400 5600
-Wire Wire Line
 	9200 5000 9500 5000
 Wire Wire Line
@@
 	8800 3050 10250 3050
 Connection ~ 8800 3050
-Wire Bus Line
-	9400 3450 9400 3500
+Wire Wire Line
+	8800 5500 9500 5500
+Text Label 7750 4200 0    50   ~ 0
+D1
+Wire Bus Line
+	6700 3450 7950 3450
+Connection ~ 7950 3450
+Wire Bus Line
+	7950 3450 8150 3450
+Wire Bus Line
+	8150 3450 9400 3450
+Connection ~ 9400 3450
+Wire Wire Line
+	7750 4900 8050 4900
+Wire Wire Line
+	8050 4900 8050 1850
+Wire Wire Line
+	8050 1850 7150 1850
+Wire Wire Line
+	7150 1300 9500 1300
+Wire Wire Line
+	9500 1300 9500 4900
+Wire Wire Line
+	9500 4900 9200 4900
+$Comp
+L parts:MSM6283 U?
+U 1 1 5FA3D387
+P 3550 4850
+F 0 "U?" V 5431 4825 50  0000 C CNN
+F 1 "MSM6283" V 5340 4825 50  0000 C CNN
+F 2 "" V 2900 5200 50  0001 C CNN
+F 3 "" V 2900 5200 50  0001 C CNN
+	1    3550 4850
+	0    -1   -1   0
+$EndComp
+Wire Wire Line
+	7950 5600 6500 5600
+Wire Wire Line
+	6500 5600 6500 4850
+Wire Wire Line
+	6500 4850 4850 4850
+Connection ~ 7950 5600
+Wire Wire Line
+	7850 5700 6400 5700
+Wire Wire Line
+	6400 5700 6400 4450
+Wire Wire Line
+	6400 4450 4850 4450
+Connection ~ 7850 5700
+Wire Wire Line
+	7750 5800 6600 5800
+Wire Wire Line
+	6600 5800 6600 3150
+Wire Wire Line
+	6600 3150 4500 3150
+Connection ~ 7750 5800
+Wire Wire Line
+	9850 5700 9700 5700
+Text Label 9700 5700 0    50   ~ 0
+A15
+Entry Wire Line
+	9700 5700 9600 5600
 Wire Bus Line
 	9400 3450 9600 3450
-Connection ~ 9400 3450
-Wire Bus Line
-	7950 3450 8150 3450
-Connection ~ 7950 3450
-Wire Wire Line
-	8800 5500 9500 5500
-Wire Bus Line
-	7950 3450 7950 4900
-Wire Bus Line
-	9400 3450 9400 4900
-Wire Bus Line
-	10850 3450 10850 4700
-Wire Bus Line
-	9600 3450 9600 5200
+Wire Wire Line
+	9850 5600 9650 5600
+Wire Wire Line
+	9650 5600 9650 5500
+Wire Wire Line
+	9650 5500 9550 5500
+Wire Wire Line
+	9550 5500 9550 5600
+Wire Wire Line
+	9550 5600 9400 5600
+Connection ~ 9400 5600
+Connection ~ 9600 3450
+Wire Bus Line
+	9600 3450 10850 3450
+Wire Bus Line
+	9400 3450 9400 4700
+Wire Bus Line
+	10850 3450 10850 4500
+Wire Bus Line
+	7950 3450 7950 4700
 Wire Bus Line
 	8150 3450 8150 5200
 Wire Bus Line
 	6700 3450 6700 5200
+Wire Bus Line
+	9600 3450 9600 5600
 $EndSCHEMATC

Commit message: 'digital'
Parts:
- added C? (x2): 10nF, symbol Device:C
- added C?: 10uF @ 16V, symbol Device:CP
- added C?: 56pF @ 50v, symbol Device:C
- added C?: 84k, symbol Device:C_Variable
- added C? (x2): C, symbol Device:C
- added C?: 100uF @ 6.3v, symbol Device:CP
- added L?: LTRIM, symbol Device:LTRIM
- added R?: 10k, symbol Device:R
Connections:
- net A0: now also U?.12 (A0)
- net A1: now also U?.14 (A1)
- net A10: now also U?.17 (A10)
- net A11: now also U?.21 (A11)
- net A12: now also U?.28 (A12)
- net A13: now also U?.27 (A13)
- net A14: now also U?.29 (A14)
- net A15: now also U?.30 (A15)
- net A2: now also U?.16 (A2)
- net A3: now also U?.18 (A3)
- net A4: now also U?.20 (A4)
- net A5: now also U?.22 (A5)
- net A6: now also U?.24 (A6)
- net A7: now also U?.26 (A7)
- net A8: now also U?.25 (A8)
- net A9: now also U?.23 (A9)
- net D0: now also U?.10 (IO0)
- net D1: now also U?.8 (IO1)
- net D2: now also U?.6 (IO2)
- net D3: now also U?.5 (IO3)
- net D4: now also U?.7 (IO4)
- net D5: now also U?.9 (IO5)
- net D6: now also U?.11 (IO6)
- net D7: now also U?.13 (IO7)
- net VA: now also U?.40 (GND), C?.1, C?.2, C?.2
- net VL2: no longer U?.1 (~RFSH), U?.1 (~RFSH)
- net ~CE: now reaches U?.15 (~CE), U?.20 (~CE), U?.20 (~CE), U?.20 (~CE)
- net ~OE: now reaches U?.19 (~OE), U?.22 (~OE), U?.22 (~OE)
- net ~WE: now reaches U?.27 (~WE), U?.27 (~WE), U?.31 (~WE)
- net at U?.1 (BGND): now also U?.98 (A.GND), C?.1
- net at U?.2 (VADC): now also U?.99 (VDAC), C?.2
- net at U?.32 (~RFSH): now also U?.1 (~RFSH), U?.1 (~RFSH)
- net at U?.33 (TIN): now also U?.34 (TC0), U?.35 (TC1), U?.36 (TOUT), U?.37 (ADCTR), U?.44 (VDD2), C?.1
- net VDD1: now reaches U?.42 (TEST)
- net VDD1: now also U?.43 (VDD1), U?.59 (MI), C?.1, C?.1, C?.1, C?.1, C?.2, R?.2
- net at U?.57 (OSI): now also C?.2, C?.2, L?.2
- net at U?.58 (OSO): now also C?.2, L?.1
- net at U?.60 (RESET): now also R?.1
- net KO15: now reaches U?.61 (KO15)
- net KO9: now reaches U?.67 (KO9)
- net KO8: now reaches U?.68 (KO8)
- net KO7: now reaches U?.69 (KO7)
- net KO6: now reaches U?.70 (KO6)
- net KO5: now reaches U?.71 (KO5)
- net KO4: now reaches U?.72 (KO4)
- net KO3: now reaches U?.73 (KO3)
- net KO2: now reaches U?.74 (KO2)
- net KO1: now reaches U?.75 (KO1)
- net KO0: now reaches U?.76 (KO0)
- net KI1: now reaches U?.77 (KI1)
- net KI2: now reaches U?.78 (KI2)
- net KI3: now reaches U?.79 (KI3)
- net KI4: now reaches U?.80 (KI4)
- net KI5: now reaches U?.81 (KI5)
- net KI6: now reaches U?.82 (KI6)
- net KI7: now reaches U?.83 (KI7)
- net KI8: now reaches U?.84 (KI8)
- net AP0: now reaches U?.86 (PO1)
- net PO3: now reaches U?.88 (PO3)
- net EH: now reaches U?.89 (EH)
- net EG: now reaches U?.90 (EG)
- net EF: now reaches U?.91 (EF)
- net EE: now reaches U?.92 (EE)
- net SH: now reaches U?.93 (SH)
- net SG: now reaches U?.94 (SG)
- net SF: now reaches U?.95 (SF)
- net SE: now reaches U?.96 (SE)
- net SO: now reaches U?.97 (SO)
- new net: C?.1, C?.2
- no-connect marks 1 -> 25
