File: kicad/digital.sch (KiCad schematic (older format))
At the start: 23 parts

Commit message: 'a'
Connections:
- net AP0 renamed APO
Changed lines of the file:
@@
 $Descr A4 11693 8268
 encoding utf-8
-Sheet 4 10
+Sheet 4 11
 Title ""
 Date ""
@@
 	6700 5200 6800 5300
 Connection ~ 8150 3450
-Text Label 6800 6000 0    50   ~ 0
-VL2
-Wire Wire Line
-	6800 6000 7350 6000
 Wire Wire Line
 	10250 6000 10250 5900
@@
 Wire Wire Line
 	7350 5500 7350 6000
-Text Label 6800 3350 0    50   ~ 0
-VA
-Text Label 6800 3050 0    50   ~ 0
-VL2
-Wire Wire Line
-	6800 3350 7350 3350
 Wire Wire Line
 	10250 3350 10250 3700
@@
 Connection ~ 10250 3350
 Wire Wire Line
-	6800 3050 7350 3050
-Connection ~ 7350 3050
-Wire Wire Line
 	7350 3050 7950 3050
 $Comp
@@
 Wire Wire Line
 	7350 6000 8800 6000
-Connection ~ 7350 6000
 Wire Wire Line
 	8800 6000 10250 6000
@@
 Text HLabel 3300 6450 3    50   Output ~ 0
 PO3
-Text HLabel 3100 6450 3    50   Input ~ 0
-AP0
+Text HLabel 3100 6450 3    50   Output ~ 0
+APO
 Wire Wire Line
 	5150 6150 5150 6450
@@
 Wire Wire Line
 	3300 2900 3100 2900
+Wire Wire Line
+	2050 3100 2050 3000
+Wire Wire Line
+	3100 2900 3100 3000
+Wire Wire Line
+	3100 3000 2050 3000
+Text HLabel 7100 3050 0    50   Input ~ 0
+VL2
+Text HLabel 7100 3350 0    50   Input ~ 0
+VA
+Wire Wire Line
+	7100 3350 7350 3350
+Wire Wire Line
+	7350 3050 7100 3050
+Connection ~ 7350 3050
+Wire Wire Line
+	10250 6000 11050 6000
+Wire Wire Line
+	11050 6000 11050 3050
+Wire Wire Line
+	11050 3050 10250 3050
+Wire Bus Line
+	7950 3450 7950 5200
+Wire Bus Line
+	9400 3450 9400 5200
+Wire Bus Line
+	10850 3450 10850 4500
+Wire Bus Line
+	8150 3450 8150 5200
+Wire Bus Line
+	6700 3450 6700 5200
+Wire Bus Line
+	9600 3450 9600 5600
 Wire Bus Line
 	5100 3250 5100 5950
-Wire Bus Line
-	6700 3450 6700 5200
-Wire Bus Line
-	7950 3450 7950 5200
-Wire Bus Line
-	8150 3450 8150 5200
-Wire Bus Line
-	9400 3450 9400 5200
-Wire Bus Line
-	10850 3450 10850 4500
-Wire Bus Line
-	9600 3450 9600 5600
-Wire Wire Line
-	2050 3100 2050 3000
-Wire Wire Line
-	3100 2900 3100 3000
-Wire Wire Line
-	3100 3000 2050 3000
+Connection ~ 10250 6000
+Connection ~ 10250 3050
 $EndSCHEMATC

Commit message: 'a'
Parts:
- gave numbers to parts that had none: 19
Changed lines of the file:
@@
 $EndDescr
 $Comp
-L 74xx:74HC02 U?
+L 74xx:74HC02 U2
 U 1 1 5F82F6C9
 P 6850 1850
-F 0 "U?" H 6850 2175 50  0000 C CNN
+F 0 "U2" H 6850 2175 50  0000 C CNN
 F 1 "74HC02" H 6850 2084 50  0000 C CNN
 F 2 "" H 6850 1850 50  0001 C CNN
@@
 $EndComp
 $Comp
-L 74xx:74HC02 U?
+L 74xx:74HC02 U2
 U 2 1 5F830A6F
 P 5950 1950
-F 0 "U?" H 5950 2275 50  0000 C CNN
+F 0 "U2" H 5950 2275 50  0000 C CNN
 F 1 "74HC02" H 5950 2184 50  0000 C CNN
 F 2 "" H 5950 1950 50  0001 C CNN
@@
 $EndComp
 $Comp
-L 74xx:74HC02 U?
+L 74xx:74HC02 U2
 U 3 1 5F8318F2
 P 5950 1200
-F 0 "U?" H 5950 1525 50  0000 C CNN
+F 0 "U2" H 5950 1525 50  0000 C CNN
 F 1 "74HC02" H 5950 1434 50  0000 C CNN
 F 2 "" H 5950 1200 50  0001 C CNN
@@
 $EndComp
 $Comp
-L 74xx:74HC02 U?
+L 74xx:74HC02 U2
 U 4 1 5F832C89
 P 6850 1300
-F 0 "U?" H 6850 1625 50  0000 C CNN
+F 0 "U2" H 6850 1625 50  0000 C CNN
 F 1 "74HC02" H 6850 1534 50  0000 C CNN
 F 2 "" H 6850 1300 50  0001 C CNN
@@
 $EndComp
 $Comp
-L 74xx:74HC02 U?
+L 74xx:74HC02 U2
 U 5 1 5F834A48
 P 6350 2450
-F 0 "U?" V 6717 2450 50  0000 C CNN
+F 0 "U2" V 6717 2450 50  0000 C CNN
 F 1 "74HC02" V 6626 2450 50  0000 C CNN
 F 2 "" H 6350 2450 50  0001 C CNN
@@
 Chip Select
 $Comp
-L Memory_EPROM:27C256 U?
+L Memory_EPROM:27C256 U5
 U 1 1 5F82BB6B
 P 10250 4800
-F 0 "U?" H 10250 6081 50  0000 C CNN
+F 0 "U5" H 10250 6081 50  0000 C CNN
 F 1 "27C256" H 10250 5990 50  0000 C CNN
 F 2 "Package_DIP:DIP-28_W15.24mm" H 10250 4800 50  0001 C CNN
@@
 	8400 5300 8250 5300
 $Comp
-L parts:D4168C U?
+L parts:D4168C U4
 U 1 1 5F86613D
 P 8750 4600
-F 0 "U?" H 8800 5481 50  0000 C CNN
+F 0 "U4" H 8800 5481 50  0000 C CNN
 F 1 "D4168C" H 8800 5390 50  0000 C CNN
 F 2 "" H 8750 4600 50  0001 C CNN
@@
 	6950 5300 6800 5300
 $Comp
-L parts:D4168C U?
+L parts:D4168C U3
 U 1 1 5F8A2313
 P 7300 4600
-F 0 "U?" H 7350 5481 50  0000 C CNN
+F 0 "U3" H 7350 5481 50  0000 C CNN
 F 1 "D4168C" H 7350 5390 50  0000 C CNN
 F 2 "" H 7300 4600 50  0001 C CNN
@@
 NoConn ~ 9850 5500
 $Comp
-L Device:C C?
+L Device:C C13
 U 1 1 5F89620F
 P 7350 3200
-F 0 "C?" H 7465 3246 50  0000 L CNN
+F 0 "C13" H 7465 3246 50  0000 L CNN
 F 1 "100nF" H 7465 3155 50  0000 L CNN
 F 2 "" H 7388 3050 50  0001 C CNN
@@
 $EndComp
 $Comp
-L Device:C C?
+L Device:C C15
 U 1 1 5F896A59
 P 8800 3200
-F 0 "C?" H 8915 3246 50  0000 L CNN
+F 0 "C15" H 8915 3246 50  0000 L CNN
 F 1 "100nF" H 8915 3155 50  0000 L CNN
 F 2 "" H 8838 3050 50  0001 C CNN
@@
 $EndComp
 $Comp
-L Device:C C?
+L Device:C C16
 U 1 1 5F89735C
 P 10250 3200
-F 0 "C?" H 10365 3246 50  0000 L CNN
+F 0 "C16" H 10365 3246 50  0000 L CNN
 F 1 "100nF" H 10365 3155 50  0000 L CNN
 F 2 "" H 10288 3050 50  0001 C CNN
@@
 	7350 3050 7950 3050
 $Comp
-L Device:CP C?
+L Device:CP C14
 U 1 1 5F89E8D2
 P 7950 3200
-F 0 "C?" H 7832 3154 50  0000 R CNN
+F 0 "C14" H 7832 3154 50  0000 R CNN
 F 1 "10uF @ 16V" H 7832 3245 50  0000 R CNN
 F 2 "" H 7988 3050 50  0001 C CNN
@@
 P 3550 4850
 AR Path="/5FA3D387" Ref="U?"  Part="1"
-AR Path="/5F82B739/5FA3D387" Ref="U?"  Part="1"
-F 0 "U?" V 2000 5950 50  0000 C CNN
+AR Path="/5F82B739/5FA3D387" Ref="U1"  Part="1"
+F 0 "U1" V 2000 5950 50  0000 C CNN
 F 1 "MSM6283" H 3550 4850 50  0000 C CNN
 F 2 "" V 2900 5200 50  0001 C CNN
@@
 	3900 2700 3900 3000
 $Comp
-L Device:C C?
+L Device:C C10
 U 1 1 5FF42A50
 P 3450 2700
-F 0 "C?" V 3198 2700 50  0000 C CNN
+F 0 "C10" V 3198 2700 50  0000 C CNN
 F 1 "10nF" V 3289 2700 50  0000 C CNN
 F 2 "" H 3488 2550 50  0001 C CNN
@@
 	3300 2900 3300 3150
 $Comp
-L Device:R R?
+L Device:R R15
 U 1 1 5FFB7D91
 P 1900 4250
-F 0 "R?" V 2015 4250 50  0000 C CNN
+F 0 "R15" V 2015 4250 50  0000 C CNN
 F 1 "10k" V 2106 4250 50  0000 C CNN
 F 2 "" V 1830 4250 50  0001 C CNN
@@
 	2050 4150 2300 4150
 $Comp
-L Device:C C?
+L Device:C C7
 U 1 1 5FFE6DB0
 P 1900 3100
-F 0 "C?" V 1648 3100 50  0000 C CNN
+F 0 "C7" V 1648 3100 50  0000 C CNN
 F 1 "56pF @ 50v" V 1739 3100 50  0000 C CNN
 F 2 "" H 1938 2950 50  0001 C CNN
@@
 Connection ~ 2050 3100
 $Comp
-L Device:C_Variable C?
+L Device:C_Variable C8
 U 1 1 5FFED5AB
 P 1900 3600
-F 0 "C?" V 2152 3600 50  0000 C CNN
+F 0 "C8" V 2152 3600 50  0000 C CNN
 F 1 "84k" V 2061 3600 50  0000 C CNN
 F 2 "" H 1900 3600 50  0001 C CNN
@@
 	2300 4050 900  4050
 $Comp
-L Device:C C?
+L Device:C C5
 U 1 1 600209BF
 P 1450 3600
-F 0 "C?" V 1400 3700 50  0000 C CNN
+F 0 "C5" V 1400 3700 50  0000 C CNN
 F 1 "C" V 1500 3700 50  0000 C CNN
 F 2 "" H 1488 3450 50  0001 C CNN
@@
 $EndComp
 $Comp
-L Device:C C?
+L Device:C C6
 U 1 1 60060128
 P 1450 3800
-F 0 "C?" V 1400 3900 50  0000 C CNN
+F 0 "C6" V 1400 3900 50  0000 C CNN
 F 1 "C" V 1500 3900 50  0000 C CNN
 F 2 "" H 1488 3650 50  0001 C CNN
@@
 	900  3100 900  4050
 $Comp
-L Device:LTRIM L?
+L Device:LTRIM L1
 U 1 1 600C248B
 P 1200 3400
-F 0 "L?" H 950 3450 50  0000 L CNN
+F 0 "L1" H 950 3450 50  0000 L CNN
 F 1 "LTRIM" H 950 3350 50  0000 L CNN
 F 2 "" H 1200 3400 50  0001 C CNN
@@
 	4300 6700 4300 6450
 $Comp
-L Device:CP C?
+L Device:CP C12
 U 1 1 6018DD56
 P 5000 6450
-F 0 "C?" V 5050 6200 50  0000 C CNN
+F 0 "C12" V 5050 6200 50  0000 C CNN
 F 1 "100uF @ 6.3v" V 4950 6000 50  0000 C CNN
 F 2 "" H 5038 6300 50  0001 C CNN
@@
 	1200 3600 1200 3800
 $Comp
-L Device:C C?
+L Device:C C11
 U 1 1 5FF42F09
 P 3750 2700
-F 0 "C?" V 3498 2700 50  0000 C CNN
+F 0 "C11" V 3498 2700 50  0000 C CNN
 F 1 "10nF" V 3589 2700 50  0000 C CNN
 F 2 "" H 3788 2550 50  0001 C CNN
@@
 $EndComp
 $Comp
-L Device:CP C?
+L Device:CP C9
 U 1 1 5FF4366D
 P 3450 2500
-F 0 "C?" V 3195 2500 50  0000 C CNN
+F 0 "C9" V 3195 2500 50  0000 C CNN
 F 1 "10uF @ 16V" V 3286 2500 50  0000 C CNN
 F 2 "" H 3488 2350 50  0001 C CNN
@@
 Wire Wire Line
 	11050 3050 10250 3050
-Wire Bus Line
-	7950 3450 7950 5200
-Wire Bus Line
-	9400 3450 9400 5200
-Wire Bus Line
-	10850 3450 10850 4500
-Wire Bus Line
-	8150 3450 8150 5200
-Wire Bus Line
-	6700 3450 6700 5200
-Wire Bus Line
-	9600 3450 9600 5600
-Wire Bus Line
-	5100 3250 5100 5950
 Connection ~ 10250 6000
 Connection ~ 10250 3050
+Wire Bus Line
+	7950 3450 7950 5200
+Wire Bus Line
+	9400 3450 9400 5200
+Wire Bus Line
+	10850 3450 10850 4500
+Wire Bus Line
+	8150 3450 8150 5200
+Wire Bus Line
+	6700 3450 6700 5200
+Wire Bus Line
+	9600 3450 9600 5600
+Wire Bus Line
+	5100 3250 5100 5950
 $EndSCHEMATC
