File: kicad/moskito.sch (KiCad schematic (older format))
At the start: 0 parts

Commit message: 'a'
Other:
- note added: "VH 7.5V\nVDD1 GND\nVL1 0V\nVL2 0V\nVA 5V\nVE 3.35V\nVC 5V\nVD 5V"
Changed lines of the file:
@@
 $Descr A4 11693 8268
 encoding utf-8
-Sheet 1 10
+Sheet 1 11
 Title ""
 Date ""
@@
 $EndSheet
 $Sheet
-S 2800 700  2450 1550
+S 2600 700  2450 1550
 U 5F82B739
 F0 "CPU / RAM" 50
 F1 "digital.sch" 50
-F2 "KO1" O L 2800 850 50
-F3 "KO2" O L 2800 900 50
-F4 "KO3" O L 2800 950 50
-F5 "KO4" O L 2800 1000 50
-F6 "KO5" O L 2800 1050 50
-F7 "KO6" O L 2800 1100 50
-F8 "KO7" O L 2800 1150 50
-F9 "KO8" O L 2800 1200 50
-F10 "KO9" O L 2800 1250 50
-F11 "KO0" O L 2800 800 50
-F12 "KI1" I L 2800 1300 50
-F13 "KI2" I L 2800 1350 50
-F14 "KI3" I L 2800 1400 50
-F15 "KI4" I L 2800 1450 50
-F16 "KI5" I L 2800 1500 50
-F17 "KI6" I L 2800 1550 50
-F18 "KI7" I L 2800 1600 50
-F19 "KI8" I L 2800 1650 50
-F20 "KO15" O L 2800 1800 50
-F21 "EH" O R 5250 1350 50
-F22 "EG" O R 5250 1200 50
-F23 "EF" O R 5250 1050 50
-F24 "EE" O R 5250 900 50
-F25 "SH" O R 5250 1400 50
-F26 "SG" O R 5250 1250 50
-F27 "SF" O R 5250 1100 50
-F28 "SE" O R 5250 950 50
-F29 "SO" O R 5250 1750 50
-F30 "PO3" O R 5250 2050 50
-F31 "AP0" I R 5250 2000 50
+F2 "KO1" O L 2600 850 50
+F3 "KO2" O L 2600 900 50
+F4 "KO3" O L 2600 950 50
+F5 "KO4" O L 2600 1000 50
+F6 "KO5" O L 2600 1050 50
+F7 "KO6" O L 2600 1100 50
+F8 "KO7" O L 2600 1150 50
+F9 "KO8" O L 2600 1200 50
+F10 "KO9" O L 2600 1250 50
+F11 "KO0" O L 2600 800 50
+F12 "KI1" I L 2600 1300 50
+F13 "KI2" I L 2600 1350 50
+F14 "KI3" I L 2600 1400 50
+F15 "KI4" I L 2600 1450 50
+F16 "KI5" I L 2600 1500 50
+F17 "KI6" I L 2600 1550 50
+F18 "KI7" I L 2600 1600 50
+F19 "KI8" I L 2600 1650 50
+F20 "KO15" O L 2600 1800 50
+F21 "EH" O R 5050 1350 50
+F22 "EG" O R 5050 1200 50
+F23 "EF" O R 5050 1050 50
+F24 "EE" O R 5050 900 50
+F25 "SH" O R 5050 1400 50
+F26 "SG" O R 5050 1250 50
+F27 "SF" O R 5050 1100 50
+F28 "SE" O R 5050 950 50
+F29 "SO" O R 5050 1750 50
+F30 "PO3" O R 5050 2050 50
+F31 "APO" O R 5050 2150 50
+F32 "VL2" I R 5050 1850 50
+F33 "VA" I R 5050 1950 50
 $EndSheet
 $Sheet
@@
 $EndSheet
 Wire Wire Line
-	5250 1400 5400 1400
+	5050 1400 5400 1400
 Wire Wire Line
 	5400 2350 5850 2350
@@
 	5700 1350 5700 950
 Wire Wire Line
-	5700 950  5250 950
+	5700 950  5050 950
 Wire Wire Line
 	5850 1250 5750 1250
@@
 	5750 1250 5750 900
 Wire Wire Line
-	5750 900  5250 900
+	5750 900  5050 900
 Wire Wire Line
 	5400 1400 5400 2350
 Wire Wire Line
-	5450 1350 5250 1350
+	5450 1350 5050 1350
 Wire Wire Line
 	5850 2250 5450 2250
@@
 	5450 2250 5450 1350
 Wire Wire Line
-	5250 1250 5500 1250
+	5050 1250 5500 1250
 Wire Wire Line
 	5500 1250 5500 1650
@@
 	7050 1600 5550 1600
 Wire Wire Line
-	5550 1200 5250 1200
+	5550 1200 5050 1200
 Wire Wire Line
 	5550 1200 5550 1600
@@
 	5600 1550 5600 1100
 Wire Wire Line
-	5600 1100 5250 1100
-Wire Wire Line
-	5250 1050 5650 1050
+	5600 1100 5050 1100
+Wire Wire Line
+	5050 1050 5650 1050
 Wire Wire Line
 	5650 1050 5650 1500
@@
 	7000 1250 7150 1250
 Wire Wire Line
-	2250 850  2800 850
-Wire Wire Line
-	2800 900  2250 900
-Wire Wire Line
-	2250 950  2800 950
-Wire Wire Line
-	2800 1000 2250 1000
-Wire Wire Line
-	2250 1050 2800 1050
-Wire Wire Line
-	2800 1100 2250 1100
-Wire Wire Line
-	2250 1150 2800 1150
-Wire Wire Line
-	2800 1200 2250 1200
-Wire Wire Line
-	2250 1500 2800 1500
-Wire Wire Line
-	2800 1550 2250 1550
-Wire Wire Line
-	2250 1600 2800 1600
-Wire Wire Line
-	2800 1650 2250 1650
-$Sheet
-S 5850 2650 1050 750
+	2250 850  2600 850
+Wire Wire Line
+	2600 900  2250 900
+Wire Wire Line
+	2250 950  2600 950
+Wire Wire Line
+	2600 1000 2250 1000
+Wire Wire Line
+	2250 1050 2600 1050
+Wire Wire Line
+	2600 1100 2250 1100
+Wire Wire Line
+	2250 1150 2600 1150
+Wire Wire Line
+	2600 1200 2250 1200
+Wire Wire Line
+	2250 1500 2600 1500
+Wire Wire Line
+	2600 1550 2250 1550
+Wire Wire Line
+	2250 1600 2600 1600
+Wire Wire Line
+	2600 1650 2250 1650
+$Sheet
+S 5600 2850 1050 750
 U 5FB1A3B4
 F0 "Mic / Line In" 50
@@
 $EndSheet
 $Sheet
-S 700  2000 1550 600
+S 750  2350 1550 600
 U 5FB1A45E
 F0 "Buttons" 50
@@
 $EndSheet
 $Sheet
-S 7100 2650 1050 850
+S 7050 2900 1050 850
 U 5FB1B134
 F0 "Audio Amp" 50
@@
 F0 "Power Supply / APO" 50
 F1 "power.sch" 50
-$EndSheet
+F2 "APO" I R 4900 2750 50
+F3 "VDD1" B R 4900 3100 50
+F4 "VA" B R 4900 3450 50
+F5 "VL2" B R 4900 3000 50
+F6 "VE" B R 4900 3550 50
+F7 "VL1" B R 4900 2900 50
+F8 "VH" B R 4900 3350 50
+$EndSheet
+Text Notes 3150 3500 0    50   ~ 0
+VH 7.5V\nVDD1 GND\nVL1 0V\nVL2 0V\nVA 5V\nVE 3.35V\nVC 5V\nVD 5V
+Wire Wire Line
+	4900 2750 5100 2750
+Wire Wire Line
+	5100 2750 5100 2150
+Wire Wire Line
+	5100 2150 5050 2150
 $EndSCHEMATC
