File: kicad/moskito.sch (KiCad schematic (older format))
At the start: 0 parts

Commit message: 'a'
Changed lines of the file:
@@
 $EndSheet
 $Sheet
-S 5850 700  1050 750
+S 6050 600  1050 750
 U 5F3D82C3
 F0 "Bass" 50
 F1 "env.sch" 50
-F2 "ENV" I L 5850 1250 50
-F3 "PITCH" I L 5850 1350 50
-F4 "VD" I L 5850 900 50
-F5 "VL1" I L 5850 800 50
-F6 "OUT" O R 6900 1100 50
-$EndSheet
+F2 "ENV" I L 6050 1150 50
+F3 "PITCH" I L 6050 1250 50
+F4 "VD" I L 6050 800 50
+F5 "VL1" I L 6050 700 50
+F6 "OUT" O R 7100 1000 50
+$EndSheet
+$Sheet
+S 6050 2000 1050 750
+U 5FA5FF52
+F0 "Melody" 50
+F1 "env.sch" 50
+F2 "ENV" I L 6050 2550 50
+F3 "PITCH" I L 6050 2650 50
+F4 "VD" I L 6050 2200 50
+F5 "VL1" I L 6050 2100 50
+F6 "OUT" O R 7100 2400 50
+$EndSheet
+$Sheet
+S 7600 2000 1050 750
+U 5FA601D6
+F0 "Obbligato" 50
+F1 "env.sch" 50
+F2 "ENV" I L 7600 2550 50
+F3 "PITCH" I L 7600 2650 50
+F4 "VD" I L 7600 2200 50
+F5 "VL1" I L 7600 2100 50
+F6 "OUT" O R 8650 2400 50
+$EndSheet
+$Sheet
+S 7600 600  1050 750
+U 5FA60472
+F0 "Chord" 50
+F1 "env.sch" 50
+F2 "ENV" I L 7600 1150 50
+F3 "PITCH" I L 7600 1250 50
+F4 "VD" I L 7600 800 50
+F5 "VL1" I L 7600 700 50
+F6 "OUT" O R 8650 1000 50
+$EndSheet
+Wire Wire Line
+	5050 1400 5350 1400
+Wire Wire Line
+	5350 2650 6050 2650
+Wire Wire Line
+	6050 1250 5800 1250
+Wire Wire Line
+	5800 1250 5800 950
+Wire Wire Line
+	5800 950  5050 950
+Wire Wire Line
+	6050 1150 5850 1150
+Wire Wire Line
+	5850 1150 5850 900
+Wire Wire Line
+	5850 900  5050 900
+Wire Wire Line
+	5350 1400 5350 2650
+Wire Wire Line
+	5400 1350 5050 1350
+Wire Wire Line
+	6050 2550 5400 2550
+Wire Wire Line
+	5400 2550 5400 1350
+Wire Wire Line
+	5050 1250 5500 1250
+Wire Wire Line
+	5500 1250 5500 1900
+Wire Wire Line
+	5500 1900 7300 1900
+Wire Wire Line
+	7300 1900 7300 2650
+Wire Wire Line
+	7300 2650 7600 2650
+Wire Wire Line
+	7600 2550 7350 2550
+Wire Wire Line
+	7350 2550 7350 1850
+Wire Wire Line
+	7350 1850 5550 1850
+Wire Wire Line
+	5550 1200 5050 1200
+Wire Wire Line
+	5550 1200 5550 1850
+Wire Wire Line
+	7600 1250 7350 1250
+Wire Wire Line
+	7350 1250 7350 1500
+Wire Wire Line
+	7350 1500 5650 1500
+Wire Wire Line
+	5650 1500 5650 1100
+Wire Wire Line
+	5650 1100 5050 1100
+Wire Wire Line
+	5050 1050 5700 1050
+Wire Wire Line
+	5700 1050 5700 1450
+Wire Wire Line
+	5700 1450 7300 1450
+Wire Wire Line
+	7300 1450 7300 1150
+Wire Wire Line
+	7300 1150 7600 1150
+Wire Wire Line
+	2250 850  2600 850
+Wire Wire Line
+	2600 900  2250 900
+Wire Wire Line
+	2250 950  2600 950
+Wire Wire Line
+	2600 1000 2250 1000
+Wire Wire Line
+	2250 1050 2600 1050
+Wire Wire Line
+	2600 1100 2250 1100
+Wire Wire Line
+	2250 1150 2600 1150
+Wire Wire Line
+	2600 1200 2250 1200
+Wire Wire Line
+	2250 1500 2600 1500
+Wire Wire Line
+	2600 1550 2250 1550
+Wire Wire Line
+	2250 1600 2600 1600
+Wire Wire Line
+	2600 1650 2250 1650
+$Sheet
+S 5800 3500 1050 750
+U 5FB1A3B4
+F0 "Mic / Line In" 50
+F1 "audioin.sch" 50
+$EndSheet
+$Sheet
+S 750  2350 1550 600
+U 5FB1A45E
+F0 "Buttons" 50
+F1 "buttons.sch" 50
+$EndSheet
+$Sheet
+S 7250 3600 1050 850
+U 5FB1B134
+F0 "Audio Amp" 50
+F1 "amp.sch" 50
+$EndSheet
+$Sheet
+S 2800 2650 2100 1100
+U 5FB1B1A6
+F0 "Power Supply / APO" 50
+F1 "power.sch" 50
+F2 "APO" I R 4900 2750 50
+F3 "VDD1" B L 2800 3550 50
+F4 "VA" B R 4900 2900 50
+F5 "VL2" B R 4900 3000 50
+F6 "VE" B L 2800 3650 50
+F7 "VL1" B R 4900 3150 50
+F8 "VH" B L 2800 3450 50
+F9 "VC" B L 2800 3700 50
+F10 "VD" B R 4900 3250 50
+$EndSheet
+Text Notes 3150 3500 0    50   ~ 0
+VH 7.5V\nVDD1 GND\nVL1 0V\nVL2 0V\nVA 5V\nVE 3.35V\nVC 5V\nVD 5V
+Wire Wire Line
+	4900 2750 5100 2750
+Wire Wire Line
+	5100 2750 5100 2150
+Wire Wire Line
+	5100 2150 5050 2150
+Wire Wire Line
+	6050 700  5950 700
+Wire Wire Line
+	5950 700  5950 1650
+Wire Wire Line
+	6050 800  6000 800
+Wire Wire Line
+	6000 800  6000 1700
+Wire Wire Line
+	7600 700  7500 700
+Wire Wire Line
+	7550 800  7600 800
+Wire Wire Line
+	5750 1650 5950 1650
+Wire Wire Line
+	5800 1700 6000 1700
+Wire Wire Line
+	7500 700  7500 1650
+Wire Wire Line
+	7500 2100 7600 2100
+Wire Wire Line
+	7600 2200 7550 2200
+Wire Wire Line
+	7550 800  7550 1700
+Wire Wire Line
+	6050 2200 6000 2200
+Wire Wire Line
+	6000 2200 6000 1700
+Connection ~ 6000 1700
+Wire Wire Line
+	6050 2100 5950 2100
+Wire Wire Line
+	5950 2100 5950 1650
+Connection ~ 5950 1650
+Wire Wire Line
+	5950 1650 7500 1650
+Connection ~ 7500 1650
+Wire Wire Line
+	7500 1650 7500 2100
+Wire Wire Line
+	7550 1700 6000 1700
+Connection ~ 7550 1700
+Wire Wire Line
+	7550 1700 7550 2200
+Wire Wire Line
+	5050 1850 5200 1850
+Wire Wire Line
+	5200 1850 5200 3000
+Wire Wire Line
+	5200 3000 4900 3000
 $Sheet
 S 2600 700  2450 1550
@@
 F33 "VA" I R 5050 1950 50
 $EndSheet
-$Sheet
-S 5850 1700 1050 750
-U 5FA5FF52
-F0 "Melody" 50
-F1 "env.sch" 50
-F2 "ENV" I L 5850 2250 50
-F3 "PITCH" I L 5850 2350 50
-F4 "VD" I L 5850 1900 50
-F5 "VL1" I L 5850 1800 50
-F6 "OUT" O R 6900 2100 50
-$EndSheet
-$Sheet
-S 7150 1700 1050 750
-U 5FA601D6
-F0 "Obbligato" 50
-F1 "env.sch" 50
-F2 "ENV" I L 7150 2250 50
-F3 "PITCH" I L 7150 2350 50
-F4 "VD" I L 7150 1900 50
-F5 "VL1" I L 7150 1800 50
-F6 "OUT" O R 8200 2100 50
-$EndSheet
-$Sheet
-S 7150 700  1050 750
-U 5FA60472
-F0 "Chord" 50
-F1 "env.sch" 50
-F2 "ENV" I L 7150 1250 50
-F3 "PITCH" I L 7150 1350 50
-F4 "VD" I L 7150 900 50
-F5 "VL1" I L 7150 800 50
-F6 "OUT" O R 8200 1100 50
-$EndSheet
-Wire Wire Line
-	5050 1400 5400 1400
-Wire Wire Line
-	5400 2350 5850 2350
-Wire Wire Line
-	5850 1350 5700 1350
-Wire Wire Line
-	5700 1350 5700 950
-Wire Wire Line
-	5700 950  5050 950
-Wire Wire Line
-	5850 1250 5750 1250
-Wire Wire Line
-	5750 1250 5750 900
-Wire Wire Line
-	5750 900  5050 900
-Wire Wire Line
-	5400 1400 5400 2350
-Wire Wire Line
-	5450 1350 5050 1350
-Wire Wire Line
-	5850 2250 5450 2250
-Wire Wire Line
-	5450 2250 5450 1350
-Wire Wire Line
-	5050 1250 5500 1250
-Wire Wire Line
-	5500 1250 5500 1650
-Wire Wire Line
-	5500 1650 7000 1650
-Wire Wire Line
-	7000 1650 7000 2350
-Wire Wire Line
-	7000 2350 7150 2350
-Wire Wire Line
-	7150 2250 7050 2250
-Wire Wire Line
-	7050 2250 7050 1600
-Wire Wire Line
-	7050 1600 5550 1600
-Wire Wire Line
-	5550 1200 5050 1200
-Wire Wire Line
-	5550 1200 5550 1600
-Wire Wire Line
-	7150 1350 7050 1350
-Wire Wire Line
-	7050 1350 7050 1550
-Wire Wire Line
-	7050 1550 5600 1550
-Wire Wire Line
-	5600 1550 5600 1100
-Wire Wire Line
-	5600 1100 5050 1100
-Wire Wire Line
-	5050 1050 5650 1050
-Wire Wire Line
-	5650 1050 5650 1500
-Wire Wire Line
-	5650 1500 7000 1500
-Wire Wire Line
-	7000 1500 7000 1250
-Wire Wire Line
-	7000 1250 7150 1250
-Wire Wire Line
-	2250 850  2600 850
-Wire Wire Line
-	2600 900  2250 900
-Wire Wire Line
-	2250 950  2600 950
-Wire Wire Line
-	2600 1000 2250 1000
-Wire Wire Line
-	2250 1050 2600 1050
-Wire Wire Line
-	2600 1100 2250 1100
-Wire Wire Line
-	2250 1150 2600 1150
-Wire Wire Line
-	2600 1200 2250 1200
-Wire Wire Line
-	2250 1500 2600 1500
-Wire Wire Line
-	2600 1550 2250 1550
-Wire Wire Line
-	2250 1600 2600 1600
-Wire Wire Line
-	2600 1650 2250 1650
-$Sheet
-S 5600 2850 1050 750
-U 5FB1A3B4
-F0 "Mic / Line In" 50
-F1 "audioin.sch" 50
-$EndSheet
-$Sheet
-S 750  2350 1550 600
-U 5FB1A45E
-F0 "Buttons" 50
-F1 "buttons.sch" 50
-$EndSheet
-$Sheet
-S 7050 2900 1050 850
-U 5FB1B134
-F0 "Audio Amp" 50
-F1 "amp.sch" 50
-$EndSheet
-$Sheet
-S 2800 2650 2100 1100
-U 5FB1B1A6
-F0 "Power Supply / APO" 50
-F1 "power.sch" 50
-F2 "APO" I R 4900 2750 50
-F3 "VDD1" B R 4900 3100 50
-F4 "VA" B R 4900 3400 50
-F5 "VL2" B R 4900 3000 50
-F6 "VE" B R 4900 3500 50
-F7 "VL1" B R 4900 2900 50
-F8 "VH" B R 4900 3300 50
-F9 "VC" B R 4900 3600 50
-F10 "VD" B R 4900 3700 50
-$EndSheet
-Text Notes 3150 3500 0    50   ~ 0
-VH 7.5V\nVDD1 GND\nVL1 0V\nVL2 0V\nVA 5V\nVE 3.35V\nVC 5V\nVD 5V
-Wire Wire Line
-	4900 2750 5100 2750
-Wire Wire Line
-	5100 2750 5100 2150
-Wire Wire Line
-	5100 2150 5050 2150
+Wire Wire Line
+	5050 1950 5150 1950
+Wire Wire Line
+	5150 1950 5150 2900
+Wire Wire Line
+	5150 2900 4900 2900
+Wire Wire Line
+	5750 3150 4900 3150
+Wire Wire Line
+	5750 1650 5750 3150
+Wire Wire Line
+	5800 3250 4900 3250
+Wire Wire Line
+	5800 1700 5800 3250
 $EndSCHEMATC

Commit message: 'a'
Changed lines of the file:
@@
 	2600 1650 2250 1650
 $Sheet
-S 5800 3500 1050 750
+S 1250 3000 1050 750
 U 5FB1A3B4
 F0 "Mic / Line In" 50
@@
 $EndSheet
 $Sheet
-S 750  2350 1550 600
+S 700  2050 1550 600
 U 5FB1A45E
 F0 "Buttons" 50
@@
 $EndSheet
 $Sheet
-S 7250 3600 1050 850
+S 9200 1150 1050 850
 U 5FB1B134
 F0 "Audio Amp" 50
@@
 $EndSheet
 $Sheet
-S 2800 2650 2100 1100
+S 2800 3200 2100 1100
 U 5FB1B1A6
 F0 "Power Supply / APO" 50
 F1 "power.sch" 50
-F2 "APO" I R 4900 2750 50
-F3 "VDD1" B L 2800 3550 50
-F4 "VA" B R 4900 2900 50
-F5 "VL2" B R 4900 3000 50
-F6 "VE" B L 2800 3650 50
-F7 "VL1" B R 4900 3150 50
-F8 "VH" B L 2800 3450 50
-F9 "VC" B L 2800 3700 50
-F10 "VD" B R 4900 3250 50
+F2 "APO" I R 4900 3300 50
+F3 "VDD1" B L 2800 4100 50
+F4 "VA" B R 4900 3450 50
+F5 "VL2" B R 4900 3550 50
+F6 "VE" B L 2800 4200 50
+F7 "VL1" B R 4900 3700 50
+F8 "VH" B L 2800 4000 50
+F9 "VC" B L 2800 4250 50
+F10 "VD" B R 4900 3800 50
 $EndSheet
-Text Notes 3150 3500 0    50   ~ 0
+Text Notes 3650 4050 0    50   ~ 0
 VH 7.5V\nVDD1 GND\nVL1 0V\nVL2 0V\nVA 5V\nVE 3.35V\nVC 5V\nVD 5V
 Wire Wire Line
-	4900 2750 5100 2750
+	4900 3300 5100 3300
 Wire Wire Line
-	5100 2750 5100 2150
+	5100 3300 5100 2150
 Wire Wire Line
 	5100 2150 5050 2150
@@
 	7550 1700 7550 2200
 Wire Wire Line
-	5050 1850 5200 1850
+	5050 1900 5200 1900
 Wire Wire Line
-	5200 1850 5200 3000
+	5200 1900 5200 3550
 Wire Wire Line
-	5200 3000 4900 3000
+	5200 3550 4900 3550
 $Sheet
 S 2600 700  2450 1550
@@
 F27 "SF" O R 5050 1100 50
 F28 "SE" O R 5050 950 50
-F29 "SO" O R 5050 1750 50
-F30 "PO3" O R 5050 2050 50
+F29 "SO" O L 2600 2050 50
+F30 "PO3" O L 2600 2150 50
 F31 "APO" O R 5050 2150 50
-F32 "VL2" I R 5050 1850 50
-F33 "VA" I R 5050 1950 50
+F32 "VL2" I R 5050 1900 50
+F33 "VA" I R 5050 2000 50
 $EndSheet
 Wire Wire Line
-	5050 1950 5150 1950
+	5050 2000 5150 2000
 Wire Wire Line
-	5150 1950 5150 2900
+	5150 2000 5150 3450
 Wire Wire Line
-	5150 2900 4900 2900
+	5150 3450 4900 3450
 Wire Wire Line
-	5750 3150 4900 3150
+	5750 3700 4900 3700
 Wire Wire Line
-	5750 1650 5750 3150
+	5750 1650 5750 3700
 Wire Wire Line
-	5800 3250 4900 3250
+	5800 3800 4900 3800
 Wire Wire Line
-	5800 1700 5800 3250
+	5800 1700 5800 3800
 $EndSCHEMATC
