File: kicad/audioin.sch (KiCad schematic (older format))
At the start: 0 parts

Commit message: 'a'
Parts:
- added MK?: Microphone_Condenser, symbol Device:Microphone_Condenser
- added Q? (x2): 2SC1740LNSR-TP-T, symbol Device:Q_NPN_BCE
Changed lines of the file:
@@
 $Descr A4 11693 8268
 encoding utf-8
-Sheet 1 11
+Sheet 7 11
 Title ""
 Date ""
@@
 Comment4 ""
 $EndDescr
+Text HLabel 1000 1100 0    50   Input ~ 0
+VL1
+Text HLabel 1000 900  0    50   Input ~ 0
+VC
+Text HLabel 1000 1300 0    50   Output ~ 0
+VIM
+$Comp
+L Device:Microphone_Condenser MK?
+U 1 1 5FAE0F72
+P 5800 1050
+F 0 "MK?" H 5930 1096 50  0000 L CNN
+F 1 "Microphone_Condenser" H 5930 1005 50  0000 L CNN
+F 2 "" V 5800 1150 50  0001 C CNN
+F 3 "~" V 5800 1150 50  0001 C CNN
+	1    5800 1050
+	1    0    0    -1
+$EndComp
+$Comp
+L Device:Q_NPN_BCE Q?
+U 1 1 5FAE1C5B
+P 4100 2350
+F 0 "Q?" V 4335 2350 50  0000 C CNN
+F 1 "2SC1740LNSR-TP-T" V 4426 2350 50  0000 C CNN
+F 2 "" H 4300 2450 50  0001 C CNN
+F 3 "~" H 4100 2350 50  0001 C CNN
+	1    4100 2350
+	0    1    1    0
+$EndComp
+$Comp
+L Device:Q_NPN_BCE Q?
+U 1 1 5FAE1FB6
+P 4500 3450
+F 0 "Q?" V 4735 3450 50  0000 C CNN
+F 1 "2SC1740LNSR-TP-T" V 4826 3450 50  0000 C CNN
+F 2 "" H 4700 3550 50  0001 C CNN
+F 3 "~" H 4500 3450 50  0001 C CNN
+	1    4500 3450
+	0    1    1    0
+$EndComp
 $EndSCHEMATC
