File: kicad/buttons.sch (KiCad schematic (older format))
At the start: 0 parts

Commit message: 'a'
Parts:
- added D?: LN251RPP.WE, symbol Device:LED
- added SW? (x2): SW_DP3T, symbol Switch:SW_DP3T
- added SW?: SW_SP4T, symbol parts:SW_SP4T
- added SW? (x27): SW_SPST, symbol Switch:SW_SPST
