File: kicad/power.sch (KiCad schematic (older format))
At the start: 19 parts

Commit message: 'a'
Parts:
- added C29: 100uF @ 6.3V, symbol Device:CP
- added C30: 220uF @ 6.3V, symbol Device:CP
- added C31, C32: 10nF, symbol Device:C
- added C33: 47uF @ 10V, symbol Device:CP
- added J2: Jack-DC, symbol Connector:Jack-DC
- added Q13: 2SC17405Q-TP-T, symbol Device:Q_NPN_BCE
- added Q16: 2SA934R, symbol Device:Q_PNP_BCE
- added R59: 100, symbol Device:R
- added R60: 33, symbol Device:R
- added R61: 100k, symbol Device:R
- added R62: 120k, symbol Device:R
- added R64, R65: 2.2k, symbol Device:R
- added R67: 10k, symbol Device:R
- gave numbers to parts that had none: 19
Connections:
- net VA: now also C32.2, C33.1, R59.1, R60.1
- net VDD1: now also C32.1, C33.2, J2.1, Q13.3 (E), R62.1
- net VH: now also C31.2, Q16.2 (C)
- net VL1: now also C29.2, C30.2, C31.1
- net at C35.1, Q20.3 (E), R74.1: now also J2.2, Q16.3 (E), R67.1
- net at Q15.2 (C), R66.1, R69.2: now also R61.1
- new net: Q16.1 (B), R64.1, R65.1, R67.2
- new net: Q13.1 (B), R61.2, R62.2
- new net: Q13.2 (C), R64.2, R65.2
- new net VC: C29.1, R59.2
- new net VD: C30.1, R60.2
Other:
- note added: "0.0V"
- note added: "0.7V"
- note added: "APO Circuit"
- moved on the sheet: C35

Commit message: 'a'
Parts:
- removed D45: LN2G, symbol Device:D
- removed J2: Jack-DC, symbol Connector:Jack-DC
- added BT?: Battery, symbol Device:Battery
- added D?: LN2G, symbol Device:LED
- added J?: Barrel_Jack_Switch, symbol Connector:Barrel_Jack_Switch
Connections:
- net VDD1: now also BT?.2 (-), D?.1 (K), J?.1
- net at C35.1, Q16.3 (E), Q20.3 (E)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: now also J?.2
- net at Q18.3 (E), R73.2: now also D?.2 (A)
- new net: BT?.1 (+), J?.3
Changed lines of the file:
@@
 $Descr A4 11693 8268
 encoding utf-8
-Sheet 11 11
+Sheet 10 11
 Title ""
 Date ""
@@
 	1    9150 2400
 	1    0    0    -1
-$EndComp
-$Comp
-L Device:D D45
-U 1 1 5FAA5D5C
-P 9250 2950
-F 0 "D45" V 9296 2870 50  0000 R CNN
-F 1 "LN2G" V 9205 2870 50  0000 R CNN
-F 2 "" H 9250 2950 50  0001 C CNN
-F 3 "~" H 9250 2950 50  0001 C CNN
-	1    9250 2950
-	0    -1   -1   0
 $EndComp
 Wire Wire Line
@@
 Wire Wire Line
 	10200 1750 10200 600
-$Comp
-L Connector:Jack-DC J2
-U 1 1 5FC229FA
-P 10950 1350
-F 0 "J2" H 11100 1550 50  0000 R CNN
-F 1 "Jack-DC" H 11100 1650 50  0000 R CNN
-F 2 "" H 11000 1310 50  0001 C CNN
-F 3 "~" H 11000 1310 50  0001 C CNN
-	1    10950 1350
-	-1   0    0    1
-$EndComp
 Wire Wire Line
 	10650 1250 10650 1100
-Wire Wire Line
-	10650 1100 10350 1100
 Connection ~ 10350 1100
 Wire Wire Line
 	10650 1450 10650 1750
 Wire Wire Line
-	10650 1750 10350 1750
+	10650 1750 10600 1750
 Connection ~ 10350 1750
 Text Notes 6100 3850 0    50   ~ 0
@@
 Text Notes 5550 2300 0    50   ~ 0
 0.7V
+$Comp
+L Device:LED D?
+U 1 1 5FAE8FBA
+P 9250 2950
+F 0 "D?" V 9289 2832 50  0000 R CNN
+F 1 "LN2G" V 9198 2832 50  0000 R CNN
+F 2 "" H 9250 2950 50  0001 C CNN
+F 3 "~" H 9250 2950 50  0001 C CNN
+	1    9250 2950
+	0    -1   -1   0
+$EndComp
+$Comp
+L Connector:Barrel_Jack_Switch J?
+U 1 1 5FAEB180
+P 10950 1350
+F 0 "J?" H 10720 1300 50  0000 R CNN
+F 1 "Barrel_Jack_Switch" H 10720 1391 50  0000 R CNN
+F 2 "" H 11000 1310 50  0001 C CNN
+F 3 "~" H 11000 1310 50  0001 C CNN
+	1    10950 1350
+	-1   0    0    1
+$EndComp
+$Comp
+L Device:Battery BT?
+U 1 1 5FAEC2E4
+P 10600 800
+F 0 "BT?" H 10708 846 50  0000 L CNN
+F 1 "Battery" H 10708 755 50  0000 L CNN
+F 2 "" V 10600 860 50  0001 C CNN
+F 3 "~" V 10600 860 50  0001 C CNN
+	1    10600 800
+	1    0    0    -1
+$EndComp
+Wire Wire Line
+	10650 1350 10500 1350
+Wire Wire Line
+	10350 1100 10650 1100
+Wire Wire Line
+	10600 600  10500 600
+Wire Wire Line
+	10500 600  10500 1350
+Wire Wire Line
+	10600 1000 10600 1750
+Connection ~ 10600 1750
+Wire Wire Line
+	10600 1750 10350 1750
 $EndSCHEMATC
