File: kicad/amp.sch (KiCad schematic (older format))
At the start: 0 parts

Commit message: 'la4138'
Parts:
- added U?: LA4138, symbol parts:LA4138
Changed lines of the file:
@@
 $Descr A4 11693 8268
 encoding utf-8
-Sheet 1 11
+Sheet 9 11
 Title ""
 Date ""
@@
 Comment4 ""
 $EndDescr
+$Comp
+L parts:LA4138 U?
+U 1 1 5FB1BF5F
+P 5200 3500
+F 0 "U?" H 5644 3571 50  0000 L CNN
+F 1 "LA4138" H 5644 3480 50  0000 L CNN
+F 2 "" H 5150 2600 50  0001 C CNN
+F 3 "" H 5150 2600 50  0001 C CNN
+	1    5200 3500
+	1    0    0    -1
+$EndComp
 $EndSCHEMATC
